Commit message: corrected some mispelled references to the package name and updated file references in the urdf

File: staubli_rx170_support/urdf/rx170.xacro (robot description, xacro)
@@ -1,5 +1,5 @@
 <?xml version="1.0" ?>
 <robot name="staubli_rx170" xmlns:xacro="http://ros.org/wiki/xacro">
-	<include filename="$(find stabuli)/rx170/urdf/rx170_macro.xacro"/>
-	<xacro:stabuli_rx170 prefix=""/>
+	<include filename="$(find staubli)/staubli_rx170_support/urdf/rx170_macro.xacro"/>
+	<xacro:staubli_rx170 prefix=""/>
 </robot>

File: staubli_rx170_support/urdf/rx170_macro.xacro (robot description, xacro)
@@ -10,5 +10,5 @@
     <collision>
       <geometry>
-        <mesh filename="package://staubli_rx170/meshes/collision/base_link_collision.dae" />
+        <mesh filename="package://staubli_rx170/meshes/collision/base_link.dae" />
       </geometry>
     </collision>
@@ -29,5 +29,5 @@
     <collision>
       <geometry>
-        <mesh filename="package://staubli_rx170/meshes/collision/shoulder_link_collision.dae" />
+        <mesh filename="package://staubli_rx170/meshes/collision/shoulder_link.dae" />
       </geometry>
     </collision>
@@ -48,5 +48,5 @@
     <collision>
       <geometry>
-        <mesh filename="package://staubli_rx170/meshes/collision/arm_link_collision.dae" />
+        <mesh filename="package://staubli_rx170/meshes/collision/arm_link.dae" />
       </geometry>
     </collision>
@@ -67,5 +67,5 @@
     <collision>
       <geometry>
-        <mesh filename="package://staubli_rx170/meshes/collision/elbow_link_collision.dae" />
+        <mesh filename="package://staubli_rx170/meshes/collision/elbow_link.dae" />
       </geometry>
     </collision>
@@ -86,5 +86,5 @@
     <collision>
       <geometry>
-        <mesh filename="package://staubli_rx170/meshes/collision/forearm_link_collision.dae" />
+        <mesh filename="package://staubli_rx170/meshes/collision/forearm_link.dae" />
       </geometry>
     </collision>
@@ -105,5 +105,5 @@
     <collision>
       <geometry>
-        <mesh filename="package://staubli_rx170/meshes/collision/wrist_link_collision.dae" />
+        <mesh filename="package://staubli_rx170/meshes/collision/wrist_link.dae" />
       </geometry>
     </collision>
@@ -124,5 +124,5 @@
     <collision>
       <geometry>
-        <mesh filename="package://staubli_rx170/meshes/collision/grinder_collision.dae" />
+        <mesh filename="package://staubli_rx170/meshes/collision/grinder.dae" />
       </geometry>
     </collision>

Commit message: added some missing package files, fixed some references in the macro.xacro, and generated the urdf

File: staubli_rx170_support/urdf/rx170.xacro (robot description, xacro)
@@ -1,5 +1,5 @@
 <?xml version="1.0" ?>
 <robot name="staubli_rx170" xmlns:xacro="http://ros.org/wiki/xacro">
-	<include filename="$(find staubli)/staubli_rx170_support/urdf/rx170_macro.xacro"/>
+	<include filename="$(find staubli_rx170_support)/urdf/rx170_macro.xacro"/>
 	<xacro:staubli_rx170 prefix=""/>
 </robot>

File: staubli_rx170_support/urdf/rx170_macro.xacro (robot description, xacro)
@@ -5,10 +5,10 @@
     <visual>
       <geometry>
-        <mesh filename="package://staubli_rx170/meshes/visual/base_link.dae" />
+        <mesh filename="package://staubli_rx170_support/meshes/visual/base_link.dae" />
       </geometry>
     </visual>
     <collision>
       <geometry>
-        <mesh filename="package://staubli_rx170/meshes/collision/base_link.dae" />
+        <mesh filename="package://staubli_rx170_support/meshes/collision/base_link.dae" />
       </geometry>
     </collision>
@@ -24,10 +24,10 @@
     <visual>
       <geometry>
-        <mesh filename="package://staubli_rx170/meshes/visual/shoulder_link.dae" />
+        <mesh filename="package://staubli_rx170_support/meshes/visual/shoulder_link.dae" />
       </geometry>
     </visual>
     <collision>
       <geometry>
-        <mesh filename="package://staubli_rx170/meshes/collision/shoulder_link.dae" />
+        <mesh filename="package://staubli_rx170_support/meshes/collision/shoulder_link.dae" />
       </geometry>
     </collision>
@@ -43,10 +43,10 @@
     <visual>
       <geometry>
-        <mesh filename="package://staubli_rx170/meshes/visual/arm_link.dae" />
+        <mesh filename="package://staubli_rx170_support/meshes/visual/arm_link.dae" />
       </geometry>
     </visual>
     <collision>
       <geometry>
-        <mesh filename="package://staubli_rx170/meshes/collision/arm_link.dae" />
+        <mesh filename="package://staubli_rx170_support/meshes/collision/arm_link.dae" />
       </geometry>
     </collision>
@@ -62,10 +62,10 @@
     <visual>
       <geometry>
-        <mesh filename="package://staubli_rx170/meshes/visual/elbow_link.dae" />
+        <mesh filename="package://staubli_rx170_support/meshes/visual/elbow_link.dae" />
       </geometry>
     </visual>
     <collision>
       <geometry>
-        <mesh filename="package://staubli_rx170/meshes/collision/elbow_link.dae" />
+        <mesh filename="package://staubli_rx170_support/meshes/collision/elbow_link.dae" />
       </geometry>
     </collision>
@@ -81,10 +81,10 @@
     <visual>
       <geometry>
-        <mesh filename="package://staubli_rx170/meshes/visual/forearm_link.dae" />
+        <mesh filename="package://staubli_rx170_support/meshes/visual/forearm_link.dae" />
       </geometry>
     </visual>
     <collision>
       <geometry>
-        <mesh filename="package://staubli_rx170/meshes/collision/forearm_link.dae" />
+        <mesh filename="package://staubli_rx170_support/meshes/collision/forearm_link.dae" />
       </geometry>
     </collision>
@@ -100,10 +100,10 @@
     <visual>
       <geometry>
-        <mesh filename="package://staubli_rx170/meshes/visual/wrist_link.dae" />
+        <mesh filename="package://staubli_rx170_support/meshes/visual/wrist_link.dae" />
       </geometry>
     </visual>
     <collision>
       <geometry>
-        <mesh filename="package://staubli_rx170/meshes/collision/wrist_link.dae" />
+        <mesh filename="package://staubli_rx170_support/meshes/collision/wrist_link.dae" />
       </geometry>
     </collision>
@@ -119,10 +119,10 @@
     <visual>
       <geometry>
-        <mesh filename="package://staubli_rx170/meshes/visual/grinder.dae" />
+        <mesh filename="package://staubli_rx170_support/meshes/visual/grinder.dae" />
       </geometry>
     </visual>
     <collision>
       <geometry>
-        <mesh filename="package://staubli_rx170/meshes/collision/grinder.dae" />
+        <mesh filename="package://staubli_rx170_support/meshes/collision/grinder.dae" />
       </geometry>
     </collision>
