Commit message: rx160: fix spaces vs tabs in RX160L xacro macro.

File: staubli_rx160_support/urdf/rx160l_macro.xacro (robot description, xacro)
@@ -68,5 +68,5 @@
 				<origin xyz="0 0 0" rpy="0 0 0"/>
 				<geometry>
-				    <mesh filename="package://staubli_rx160_support/meshes/rx160l/visual/link_4.stl"/>
+					<mesh filename="package://staubli_rx160_support/meshes/rx160l/visual/link_4.stl"/>
 				</geometry>
 				<xacro:material_staubli_yellow />
