Commit message: Updated rx160 support package and removed deprecated syntax

File: staubli_rx160_support/urdf/rx160.xacro (robot description, xacro)
@@ -1,4 +1,4 @@
 <?xml version="1.0" ?>
-<robot name="staubli_rx160" xmlns:xacro="http://ros.org/wiki/xacro">
+<robot name="staubli_rx160" xmlns:xacro="http://wiki.ros.org/xacro">
   <xacro:include filename="$(find staubli_rx160_support)/urdf/rx160_macro.xacro"/>
   <xacro:staubli_rx160 prefix=""/>

File: staubli_rx160_support/urdf/rx160_macro.xacro (robot description, xacro)
@@ -1,7 +1,7 @@
 <?xml version="1.0"?>
-<robot xmlns:xacro="http://ros.org/wiki/xacro">
+<robot xmlns:xacro="http://wiki.ros.org/xacro">
   <xacro:include filename="$(find staubli_resources)/urdf/common_materials.xacro"/>
   <xacro:macro name="staubli_rx160" params="prefix">
-    <!-- links -->
+    <!-- links: main serial chain -->
     <link name="${prefix}base_link">
       <visual>
@@ -158,6 +158,5 @@
       </inertial>
     </link>
-    <link name="${prefix}tool0"/>
-    <!-- joints -->
+    <!-- joints: main serial chain -->
     <joint name="${prefix}joint_1" type="revolute">
       <origin xyz="0 0 0.55" rpy="0 0 0"/>
@@ -165,5 +164,5 @@
       <child link="${prefix}link_1"/>
       <axis xyz="0 0 1"/>
-      <limit lower="-2.967060" upper="2.967060" effort="692.0" velocity="2.88" />
+      <limit lower="${radians(-160)}" upper="${radians(160)}" effort="692.0" velocity="${radians(200)}" />
       <dynamics damping="0.0" friction="0.0"/>
     </joint>
@@ -173,5 +172,5 @@
       <child link="${prefix}link_2"/>
       <axis xyz="0 1 0"/>
-      <limit lower="-2.4" upper="2.4" effort="574.0" velocity="2.62" />
+      <limit lower="${radians(-137.5)}" upper="${radians(137.5)}" effort="574.0" velocity="${radians(200)}" />
       <dynamics damping="0.0" friction="0.0"/>
     </joint>
@@ -181,5 +180,5 @@
       <child link="${prefix}link_3"/>
       <axis xyz="0 1 0"/>
-      <limit lower="-2.62" upper="2.62" effort="242.0" velocity="3.32" />
+      <limit lower="${radians(-150)}" upper="${radians(150)}" effort="242.0" velocity="${radians(255)}" />
       <dynamics damping="0.0" friction="0.0"/>
     </joint>
@@ -189,5 +188,5 @@
       <child link="${prefix}link_4"/>
       <axis xyz="0 0 1"/>
-      <limit lower="-4.71" upper="4.71" effort="58.0" velocity="5.15" />
+      <limit lower="${radians(-270)}" upper="${radians(270)}" effort="58.0" velocity="${radians(315)}" />
       <dynamics damping="0.0" friction="0.0"/>
     </joint>
@@ -200,5 +199,5 @@
       (1) effort limit = 58 Nm if axis 6 torque = 0 Nm
       (2) effort limit = 29 Nm for maximum torque on axis 6 -->
-      <limit lower="-1.83" upper="2.09" effort="29.0" velocity="4.54" />
+      <limit lower="${radians(-105)}" upper="${radians(120)}" effort="29.0" velocity="${radians(360)}" />
       <dynamics damping="0.0" friction="0.0"/>
     </joint>
@@ -208,5 +207,5 @@
       <child link="${prefix}link_6"/>
       <axis xyz="0 0 1"/>
-      <limit lower="-4.71" upper="4.71" effort="29.0" velocity="7.68" />
+      <limit lower="${radians(-270)}" upper="${radians(270)}" effort="29.0" velocity="${radians(870)}" />
       <dynamics damping="0.0" friction="0.0"/>
     </joint>
@@ -216,4 +215,25 @@
       <origin xyz="0 0 0" rpy="0 0 0"/>
     </joint>
+    <!-- ROS-Industrial 'base' frame: base_link to Staubli World Coordinates transform -->
+    <link name="${prefix}base" />
+    <joint name="${prefix}base_link-base" type="fixed">
+      <origin xyz="0 0 0.550" rpy="0 0 0"/>
+      <parent link="${prefix}base_link"/>
+      <child link="${prefix}base"/>
+    </joint>
+    <!-- ROS-Industrial 'flange' frame: attachment point for EEF models -->
+    <link name="${prefix}flange" />
+    <joint name="${prefix}joint_6-flange" type="fixed">
+      <origin xyz="0 0 0" rpy="0 ${radians(-90.0)} 0" />
+      <parent link="${prefix}link_6" />
+      <child link="${prefix}flange" />
+    </joint>
+    <!-- ROS-Industrial 'tool0' frame: all-zeros tool frame -->
+    <link name="${prefix}tool0" />
+    <joint name="${prefix}flange-tool0" type="fixed">
+      <origin xyz="0 0 0" rpy="0 ${radians(90.0)} 0" />
+      <parent link="${prefix}flange" />
+      <child link="${prefix}tool0" />
+    </joint>
   </xacro:macro>
 </robot>

File: staubli_rx160_support/urdf/rx160l.xacro (robot description, xacro)
@@ -1,4 +1,4 @@
 <?xml version="1.0" ?>
-<robot name="staubli_rx160l" xmlns:xacro="http://ros.org/wiki/xacro">
+<robot name="staubli_rx160l" xmlns:xacro="http://wiki.ros.org/xacro">
   <xacro:include filename="$(find staubli_rx160_support)/urdf/rx160l_macro.xacro"/>
   <xacro:staubli_rx160l prefix=""/>

File: staubli_rx160_support/urdf/rx160l_macro.xacro (robot description, xacro)
@@ -1,7 +1,7 @@
 <?xml version="1.0"?>
-<robot xmlns:xacro="http://ros.org/wiki/xacro">
+<robot xmlns:xacro="http://wiki.ros.org/xacro">
   <xacro:include filename="$(find staubli_resources)/urdf/common_materials.xacro"/>
   <xacro:macro name="staubli_rx160l" params="prefix">
-    <!-- links -->
+    <!-- links: main serial chain -->
     <link name="${prefix}base_link">
       <visual>
@@ -158,6 +158,5 @@
       </inertial>
     </link>
-    <link name="${prefix}tool0"/>
-    <!-- joints -->
+    <!-- joints: main serial chain -->
     <joint name="${prefix}joint_1" type="revolute">
       <origin xyz="0 0 0.55" rpy="0 0 0"/>
@@ -165,5 +164,5 @@
       <child link="${prefix}link_1"/>
       <axis xyz="0 0 1"/>
-      <limit lower="-2.967060" upper="2.967060" effort="692.0" velocity="2.88" />
+      <limit lower="${radians(-160)}" upper="${radians(160)}" effort="692.0" velocity="${radians(200)}" />
       <dynamics damping="0.0" friction="0.0"/>
     </joint>
@@ -173,5 +172,5 @@
       <child link="${prefix}link_2"/>
       <axis xyz="0 1 0"/>
-      <limit lower="-2.4" upper="2.4" effort="574.0" velocity="2.62" />
+      <limit lower="${radians(-137.5)}" upper="${radians(137.5)}" effort="574.0" velocity="${radians(200)}" />
       <dynamics damping="0.0" friction="0.0"/>
     </joint>
@@ -181,5 +180,5 @@
       <child link="${prefix}link_3"/>
       <axis xyz="0 1 0"/>
-      <limit lower="-2.62" upper="2.62" effort="242.0" velocity="3.32" />
+      <limit lower="${radians(-150)}" upper="${radians(150)}" effort="242.0" velocity="${radians(255)}" />
       <dynamics damping="0.0" friction="0.0"/>
     </joint>
@@ -189,5 +188,5 @@
       <child link="${prefix}link_4"/>
       <axis xyz="0 0 1"/>
-      <limit lower="-4.71" upper="4.71" effort="58.0" velocity="5.15" />
+      <limit lower="${radians(-270)}" upper="${radians(270)}" effort="58.0" velocity="${radians(315)}" />
       <dynamics damping="0.0" friction="0.0"/>
     </joint>
@@ -200,5 +199,5 @@
       (1) effort limit = 58 Nm if axis 6 torque = 0 Nm
       (2) effort limit = 29 Nm for maximum torque on axis 6 -->
-      <limit lower="-1.83" upper="2.09" effort="29.0" velocity="4.54" />
+      <limit lower="${radians(-105)}" upper="${radians(120)}" effort="29.0" velocity="${radians(360)}" />
       <dynamics damping="0.0" friction="0.0"/>
     </joint>
@@ -208,5 +207,5 @@
       <child link="${prefix}link_6"/>
       <axis xyz="0 0 1"/>
-      <limit lower="-4.71" upper="4.71" effort="29.0" velocity="7.68" />
+      <limit lower="${radians(-270)}" upper="${radians(270)}" effort="29.0" velocity="${radians(870)}" />
       <dynamics damping="0.0" friction="0.0"/>
     </joint>
@@ -216,4 +215,25 @@
       <origin xyz="0 0 0" rpy="0 0 0"/>
     </joint>
+    <!-- ROS-Industrial 'base' frame: base_link to Staubli World Coordinates transform -->
+    <link name="${prefix}base" />
+    <joint name="${prefix}base_link-base" type="fixed">
+      <origin xyz="0 0 0.550" rpy="0 0 0"/>
+      <parent link="${prefix}base_link"/>
+      <child link="${prefix}base"/>
+    </joint>
+    <!-- ROS-Industrial 'flange' frame: attachment point for EEF models -->
+    <link name="${prefix}flange" />
+    <joint name="${prefix}joint_6-flange" type="fixed">
+      <origin xyz="0 0 0" rpy="0 ${radians(-90.0)} 0" />
+      <parent link="${prefix}link_6" />
+      <child link="${prefix}flange" />
+    </joint>
+    <!-- ROS-Industrial 'tool0' frame: all-zeros tool frame -->
+    <link name="${prefix}tool0" />
+    <joint name="${prefix}flange-tool0" type="fixed">
+      <origin xyz="0 0 0" rpy="0 ${radians(90.0)} 0" />
+      <parent link="${prefix}flange" />
+      <child link="${prefix}tool0" />
+    </joint>
   </xacro:macro>
 </robot>
