Commit message: rx160: fix link_6 mesh origin.

File: staubli_rx160_support/urdf/rx160_macro.xacro (robot description, xacro)
@@ -96,6 +96,5 @@
 		<link name="${prefix}link_6">
 			<visual>
-				<!-- TODO: fix origin of link_6 STL -->
-				<origin xyz="-0.0325 -0.0325 -0.015" rpy="0 0 0"/>
+				<origin xyz="0 0 0" rpy="0 0 0"/>
 				<geometry>
 					<mesh filename="package://staubli_rx160_support/meshes/rx160/visual/link_6.stl"/>
@@ -104,6 +103,5 @@
 			</visual>
 			<collision>
-				<!-- TODO: fix origin of link_6 STL -->
-				<origin xyz="-0.0325 -0.0325 -0.015" rpy="0 0 0"/>
+				<origin xyz="0 0 0" rpy="0 0 0"/>
 				<geometry>
 					<mesh filename="package://staubli_rx160_support/meshes/rx160/collision/link_6.stl"/>

Commit message: j6->tool0 was duplicate
as also j6->flange->tool0 exists

File: staubli_rx160_support/urdf/rx160_macro.xacro (robot description, xacro)
@@ -210,9 +210,4 @@
       <dynamics damping="0.0" friction="0.0"/>
     </joint>
-    <joint name="${prefix}joint_6-tool0" type="fixed">
-      <parent link="${prefix}link_6"/>
-      <child link="${prefix}tool0"/>
-      <origin xyz="0 0 0" rpy="0 0 0"/>
-    </joint>
     <!-- ROS-Industrial 'base' frame: base_link to Staubli World Coordinates transform -->
     <link name="${prefix}base" />

File: staubli_rx160_support/urdf/rx160l_macro.xacro (robot description, xacro)
@@ -210,9 +210,4 @@
       <dynamics damping="0.0" friction="0.0"/>
     </joint>
-    <joint name="${prefix}joint_6-tool0" type="fixed">
-      <parent link="${prefix}link_6"/>
-      <child link="${prefix}tool0"/>
-      <origin xyz="0 0 0" rpy="0 0 0"/>
-    </joint>
     <!-- ROS-Industrial 'base' frame: base_link to Staubli World Coordinates transform -->
     <link name="${prefix}base" />
