Commit message: all: fix indent to follow ROS styleguide. Fix #9.

File: staubli_rx160_support/urdf/rx160l_macro.xacro (robot description, xacro)
@@ -1,161 +1,161 @@
 <?xml version="1.0"?>
 <robot xmlns:xacro="http://ros.org/wiki/xacro">
-	<xacro:include filename="$(find staubli_resources)/urdf/common_materials.xacro"/>
-	<xacro:macro name="staubli_rx160l" params="prefix">
-		<!-- links -->
-		<link name="${prefix}base_link">
-			<visual>
-				<origin xyz="0 0 0" rpy="0 0 0"/>
-				<geometry>
-					<mesh filename="package://staubli_rx160_support/meshes/rx160/visual/base_link.stl"/>
-				</geometry>
-				<xacro:material_staubli_yellow />
-			</visual>
-			<collision>
-				<origin xyz="0 0 0" rpy="0 0 0"/>
-				<geometry>
-					<mesh filename="package://staubli_rx160_support/meshes/rx160/collision/base_link.stl"/>
-				</geometry>
-			</collision>
-		</link>
-		<link name="${prefix}link_1">
-			<visual>
-				<origin xyz="0 0 0" rpy="0 0 0"/>
-				<geometry>
-					<mesh filename="package://staubli_rx160_support/meshes/rx160/visual/link_1.stl"/>
-				</geometry>
-				<xacro:material_staubli_yellow />
-			</visual>
-			<collision>
-				<origin xyz="0 0 0" rpy="0 0 0"/>
-				<geometry>
-					<mesh filename="package://staubli_rx160_support/meshes/rx160/collision/link_1.stl"/>
-				</geometry>
-			</collision>
-		</link>
-		<link name="${prefix}link_2">
-			<visual>
-				<origin xyz="0 0 0" rpy="0 0 0"/>
-				<geometry>
-					<mesh filename="package://staubli_rx160_support/meshes/rx160/visual/link_2.stl"/>
-				</geometry>
-				<xacro:material_staubli_yellow />
-			</visual>
-			<collision>
-				<origin xyz="0 0 0" rpy="0 0 0"/>
-				<geometry>
-					<mesh filename="package://staubli_rx160_support/meshes/rx160/collision/link_2.stl"/>
-				</geometry>
-			</collision>
-		</link>
-		<link name="${prefix}link_3">
-			<visual>
-				<origin xyz="0 0 0" rpy="0 0 0"/>
-				<geometry>
-					<mesh filename="package://staubli_rx160_support/meshes/rx160/visual/link_3.stl"/>
-				</geometry>
-				<xacro:material_staubli_yellow />
-			</visual>
-			<collision>
-				<origin xyz="0 0 0" rpy="0 0 0"/>
-				<geometry>
-					<mesh filename="package://staubli_rx160_support/meshes/rx160/collision/link_3.stl"/>
-				</geometry>
-			</collision>
-		</link>
-		<link name="${prefix}link_4">
-			<visual>
-				<origin xyz="0 0 0" rpy="0 0 0"/>
-				<geometry>
-					<mesh filename="package://staubli_rx160_support/meshes/rx160l/visual/link_4.stl"/>
-				</geometry>
-				<xacro:material_staubli_yellow />
-			</visual>
-			<collision>
-				<origin xyz="0 0 0" rpy="0 0 0"/>
-				<geometry>
-					<mesh filename="package://staubli_rx160_support/meshes/rx160l/collision/link_4.stl"/>
-				</geometry>
-			</collision>
-		</link>
-		<link name="${prefix}link_5">
-			<visual>
-				<origin xyz="0 0 0" rpy="0 0 0"/>
-				<geometry>
-					<mesh filename="package://staubli_rx160_support/meshes/rx160/visual/link_5.stl"/>
-				</geometry>
-				<xacro:material_staubli_yellow />
-			</visual>
-			<collision>
-				<origin xyz="0 0 0" rpy="0 0 0"/>
-				<geometry>
-					<mesh filename="package://staubli_rx160_support/meshes/rx160/collision/link_5.stl"/>
-				</geometry>
-			</collision>
-		</link>
-		<link name="${prefix}link_6">
-			<visual>
-				<origin xyz="0 0 0" rpy="0 0 0"/>
-				<geometry>
-					<mesh filename="package://staubli_rx160_support/meshes/rx160/visual/link_6.stl"/>
-				</geometry>
-				<xacro:material_staubli_yellow />
-			</visual>
-			<collision>
-				<origin xyz="0 0 0" rpy="0 0 0"/>
-				<geometry>
-					<mesh filename="package://staubli_rx160_support/meshes/rx160/collision/link_6.stl"/>
-				</geometry>
-			</collision>
-		</link>
-		<link name="${prefix}tool0"/>
-		<!-- joints -->
-		<joint name="${prefix}joint_1" type="revolute">
-			<origin xyz="0 0 0.55" rpy="0 0 0"/>
-			<parent link="${prefix}base_link"/>
-			<child link="${prefix}link_1"/>
-			<axis xyz="0 0 1"/>
-			<limit lower="-2.967060" upper="2.967060" effort="0" velocity="2.88" />
-		</joint>
-		<joint name="${prefix}joint_2" type="revolute">
-			<origin xyz="0.15 0 0" rpy="0 0 0"/>
-			<parent link="${prefix}link_1"/>
-			<child link="${prefix}link_2"/>
-			<axis xyz="0 1 0"/>
-			<limit lower="-2.4" upper="2.4" effort="0" velocity="2.62" />
-		</joint>
-		<joint name="${prefix}joint_3" type="revolute">
-			<origin xyz="0 0 0.825" rpy="0 0 0"/>
-			<parent link="${prefix}link_2"/>
-			<child link="${prefix}link_3"/>
-			<axis xyz="0 1 0"/>
-			<limit lower="-2.62" upper="2.62" effort="0" velocity="3.32" />
-		</joint>
-		<joint name="${prefix}joint_4" type="revolute">
-			<origin xyz="0 0 0" rpy="0 0 0"/>
-			<parent link="${prefix}link_3"/>
-			<child link="${prefix}link_4"/>
-			<axis xyz="0 0 1"/>
-			<limit lower="-4.71" upper="4.71" effort="0" velocity="5.15" />
-		</joint>
-		<joint name="${prefix}joint_5" type="revolute">
-			<origin xyz="0 0 0.925" rpy="0 0 0"/>
-			<parent link="${prefix}link_4"/>
-			<child link="${prefix}link_5"/>
-			<axis xyz="0 1 0"/>
-			<limit lower="-1.83" upper="2.09" effort="0" velocity="4.54" />
-		</joint>
-		<joint name="${prefix}joint_6" type="revolute">
-			<origin xyz="0 0 0.11" rpy="0 0 0"/>
-			<parent link="${prefix}link_5"/>
-			<child link="${prefix}link_6"/>
-			<axis xyz="0 0 1"/>
-			<limit lower="-4.71" upper="4.71" effort="0" velocity="7.68" />
-		</joint>
-		<joint name="${prefix}joint_6-tool0" type="fixed">
-			<parent link="${prefix}link_6"/>
-			<child link="${prefix}tool0"/>
-			<origin xyz="0 0 0" rpy="0 0 0"/>
-		</joint>
-	</xacro:macro>
+  <xacro:include filename="$(find staubli_resources)/urdf/common_materials.xacro"/>
+  <xacro:macro name="staubli_rx160l" params="prefix">
+    <!-- links -->
+    <link name="${prefix}base_link">
+      <visual>
+        <origin xyz="0 0 0" rpy="0 0 0"/>
+        <geometry>
+          <mesh filename="package://staubli_rx160_support/meshes/rx160/visual/base_link.stl"/>
+        </geometry>
+        <xacro:material_staubli_yellow />
+      </visual>
+      <collision>
+        <origin xyz="0 0 0" rpy="0 0 0"/>
+        <geometry>
+          <mesh filename="package://staubli_rx160_support/meshes/rx160/collision/base_link.stl"/>
+        </geometry>
+      </collision>
+    </link>
+    <link name="${prefix}link_1">
+      <visual>
+        <origin xyz="0 0 0" rpy="0 0 0"/>
+        <geometry>
+          <mesh filename="package://staubli_rx160_support/meshes/rx160/visual/link_1.stl"/>
+        </geometry>
+        <xacro:material_staubli_yellow />
+      </visual>
+      <collision>
+        <origin xyz="0 0 0" rpy="0 0 0"/>
+        <geometry>
+          <mesh filename="package://staubli_rx160_support/meshes/rx160/collision/link_1.stl"/>
+        </geometry>
+      </collision>
+    </link>
+    <link name="${prefix}link_2">
+      <visual>
+        <origin xyz="0 0 0" rpy="0 0 0"/>
+        <geometry>
+          <mesh filename="package://staubli_rx160_support/meshes/rx160/visual/link_2.stl"/>
+        </geometry>
+        <xacro:material_staubli_yellow />
+      </visual>
+      <collision>
+        <origin xyz="0 0 0" rpy="0 0 0"/>
+        <geometry>
+          <mesh filename="package://staubli_rx160_support/meshes/rx160/collision/link_2.stl"/>
+        </geometry>
+      </collision>
+    </link>
+    <link name="${prefix}link_3">
+      <visual>
+        <origin xyz="0 0 0" rpy="0 0 0"/>
+        <geometry>
+          <mesh filename="package://staubli_rx160_support/meshes/rx160/visual/link_3.stl"/>
+        </geometry>
+        <xacro:material_staubli_yellow />
+      </visual>
+      <collision>
+        <origin xyz="0 0 0" rpy="0 0 0"/>
+        <geometry>
+          <mesh filename="package://staubli_rx160_support/meshes/rx160/collision/link_3.stl"/>
+        </geometry>
+      </collision>
+    </link>
+    <link name="${prefix}link_4">
+      <visual>
+        <origin xyz="0 0 0" rpy="0 0 0"/>
+        <geometry>
+          <mesh filename="package://staubli_rx160_support/meshes/rx160l/visual/link_4.stl"/>
+        </geometry>
+        <xacro:material_staubli_yellow />
+      </visual>
+      <collision>
+        <origin xyz="0 0 0" rpy="0 0 0"/>
+        <geometry>
+          <mesh filename="package://staubli_rx160_support/meshes/rx160l/collision/link_4.stl"/>
+        </geometry>
+      </collision>
+    </link>
+    <link name="${prefix}link_5">
+      <visual>
+        <origin xyz="0 0 0" rpy="0 0 0"/>
+        <geometry>
+          <mesh filename="package://staubli_rx160_support/meshes/rx160/visual/link_5.stl"/>
+        </geometry>
+        <xacro:material_staubli_yellow />
+      </visual>
+      <collision>
+        <origin xyz="0 0 0" rpy="0 0 0"/>
+        <geometry>
+          <mesh filename="package://staubli_rx160_support/meshes/rx160/collision/link_5.stl"/>
+        </geometry>
+      </collision>
+    </link>
+    <link name="${prefix}link_6">
+      <visual>
+        <origin xyz="0 0 0" rpy="0 0 0"/>
+        <geometry>
+          <mesh filename="package://staubli_rx160_support/meshes/rx160/visual/link_6.stl"/>
+        </geometry>
+        <xacro:material_staubli_yellow />
+      </visual>
+      <collision>
+        <origin xyz="0 0 0" rpy="0 0 0"/>
+        <geometry>
+          <mesh filename="package://staubli_rx160_support/meshes/rx160/collision/link_6.stl"/>
+        </geometry>
+      </collision>
+    </link>
+    <link name="${prefix}tool0"/>
+    <!-- joints -->
+    <joint name="${prefix}joint_1" type="revolute">
+      <origin xyz="0 0 0.55" rpy="0 0 0"/>
+      <parent link="${prefix}base_link"/>
+      <child link="${prefix}link_1"/>
+      <axis xyz="0 0 1"/>
+      <limit lower="-2.967060" upper="2.967060" effort="0" velocity="2.88" />
+    </joint>
+    <joint name="${prefix}joint_2" type="revolute">
+      <origin xyz="0.15 0 0" rpy="0 0 0"/>
+      <parent link="${prefix}link_1"/>
+      <child link="${prefix}link_2"/>
+      <axis xyz="0 1 0"/>
+      <limit lower="-2.4" upper="2.4" effort="0" velocity="2.62" />
+    </joint>
+    <joint name="${prefix}joint_3" type="revolute">
+      <origin xyz="0 0 0.825" rpy="0 0 0"/>
+      <parent link="${prefix}link_2"/>
+      <child link="${prefix}link_3"/>
+      <axis xyz="0 1 0"/>
+      <limit lower="-2.62" upper="2.62" effort="0" velocity="3.32" />
+    </joint>
+    <joint name="${prefix}joint_4" type="revolute">
+      <origin xyz="0 0 0" rpy="0 0 0"/>
+      <parent link="${prefix}link_3"/>
+      <child link="${prefix}link_4"/>
+      <axis xyz="0 0 1"/>
+      <limit lower="-4.71" upper="4.71" effort="0" velocity="5.15" />
+    </joint>
+    <joint name="${prefix}joint_5" type="revolute">
+      <origin xyz="0 0 0.925" rpy="0 0 0"/>
+      <parent link="${prefix}link_4"/>
+      <child link="${prefix}link_5"/>
+      <axis xyz="0 1 0"/>
+      <limit lower="-1.83" upper="2.09" effort="0" velocity="4.54" />
+    </joint>
+    <joint name="${prefix}joint_6" type="revolute">
+      <origin xyz="0 0 0.11" rpy="0 0 0"/>
+      <parent link="${prefix}link_5"/>
+      <child link="${prefix}link_6"/>
+      <axis xyz="0 0 1"/>
+      <limit lower="-4.71" upper="4.71" effort="0" velocity="7.68" />
+    </joint>
+    <joint name="${prefix}joint_6-tool0" type="fixed">
+      <parent link="${prefix}link_6"/>
+      <child link="${prefix}tool0"/>
+      <origin xyz="0 0 0" rpy="0 0 0"/>
+    </joint>
+  </xacro:macro>
 </robot>
