Commit message: Introducing Gazebo support for RX160/RX160L

File: staubli_resources/urdf/common_colours.xacro (robot description, xacro)
@@ -1,7 +1,14 @@
 <?xml version="1.0"?>
 <robot xmlns:xacro="http://ros.org/wiki/xacro">
+  <!-- RAL 1018 -->
+  <xacro:property name="colour_staubli_ral_zinc_yellow"    value="0.973 0.953 0.208 1.0" />
   <!-- RAL 1028 -->
-  <xacro:property name="colour_staubli_yellow" value="1.0 0.608 0 1" />
+  <xacro:property name="colour_staubli_ral_melon_yellow"   value="1.0 0.608 0.0 1.0" />
+  <!-- RAL 7043 -->
+  <xacro:property name="colour_staubli_ral_traffic_grey_b" value="0.306 0.329 0.322 1.0" />
   <!-- RAL 9016 -->
-  <xacro:property name="colour_staubli_white" value="0.945 0.941 0.918 1" />
+  <xacro:property name="colour_staubli_ral_traffic_white"  value="0.965 0.965 0.965 1.0" />
+  <!-- old colour definitions, for bw-compatibility. These are DEPRECATED. -->
+  <xacro:property name="colour_staubli_yellow"             value="${colour_staubli_ral_melon_yellow}" />
+  <xacro:property name="colour_staubli_white"              value="${colour_staubli_ral_traffic_white}" />
 </robot>

File: staubli_resources/urdf/common_materials.xacro (robot description, xacro)
@@ -2,4 +2,25 @@
 <robot xmlns:xacro="http://ros.org/wiki/xacro">
   <xacro:include filename="$(find staubli_resources)/urdf/common_colours.xacro"/>
+  <xacro:macro name="material_staubli_ral_zinc_yellow">
+    <material name="">
+      <color rgba="${colour_staubli_ral_zinc_yellow}"/>
+    </material>
+  </xacro:macro>
+  <xacro:macro name="material_staubli_ral_melon_yellow">
+    <material name="">
+      <color rgba="${colour_staubli_ral_melon_yellow}"/>
+    </material>
+  </xacro:macro>
+  <xacro:macro name="material_staubli_ral_traffic_grey_b">
+    <material name="">
+      <color rgba="${colour_staubli_ral_traffic_grey_b}"/>
+    </material>
+  </xacro:macro>
+  <xacro:macro name="material_staubli_ral_traffic_white">
+    <material name="">
+      <color rgba="${colour_staubli_ral_traffic_white}"/>
+    </material>
+  </xacro:macro>
+  <!-- old material definitions, for bw-compatibility. These are DEPRECATED. -->
   <xacro:macro name="material_staubli_yellow">
     <material name="">

File: staubli_rx160_support/urdf/rx160.urdf (robot description, URDF)
Before this commit: robot staubli_rx160, 8 links, 7 joints
Links:
- link base_link: mass None -> 23.085357
- link link_1: mass None -> 45.357763
- link link_2: mass None -> 51.266495
- link link_3: mass None -> 19.754401
- link link_4: mass None -> 15.287896
- link link_5: mass None -> 0.548088
- link link_6: mass None -> 0.038484
Joints:
- joint joint_1: limit lower=-2.967060 upper=2.967060 effort=0 velocity=2.88 -> lower=-2.967060 upper=2.967060 effort=692.0 velocity=2.88
- joint joint_2: limit lower=-2.4 upper=2.4 effort=0 velocity=2.62 -> lower=-2.4 upper=2.4 effort=574.0 velocity=2.62
- joint joint_3: limit lower=-2.62 upper=2.62 effort=0 velocity=3.32 -> lower=-2.62 upper=2.62 effort=242.0 velocity=3.32
- joint joint_4: limit lower=-4.71 upper=4.71 effort=0 velocity=5.15 -> lower=-4.71 upper=4.71 effort=58.0 velocity=5.15
- joint joint_5: limit lower=-1.83 upper=2.09 effort=0 velocity=4.54 -> lower=-1.83 upper=2.09 effort=29.0 velocity=4.54
- joint joint_6: limit lower=-4.71 upper=4.71 effort=0 velocity=7.68 -> lower=-4.71 upper=4.71 effort=29.0 velocity=7.68

File: staubli_rx160_support/urdf/rx160_macro.xacro (robot description, xacro)
@@ -10,5 +10,5 @@
           <mesh filename="package://staubli_rx160_support/meshes/rx160/visual/base_link.stl"/>
         </geometry>
-        <xacro:material_staubli_yellow />
+        <xacro:material_staubli_ral_melon_yellow />
       </visual>
       <collision>
@@ -18,4 +18,11 @@
         </geometry>
       </collision>
+      <inertial>
+          <mass value="23.085357"/>
+          <origin xyz="0.007579 0.000017 0.180670" rpy="0.0 0.0 0.0"/>
+          <inertia ixx="0.343576" ixy="-0.000062" ixz="-0.002079"
+                                  iyy="0.336217"  iyz="-0.000014"
+                                                  izz="0.334050"/>
+      </inertial>
     </link>
     <link name="${prefix}link_1">
@@ -25,5 +32,5 @@
           <mesh filename="package://staubli_rx160_support/meshes/rx160/visual/link_1.stl"/>
         </geometry>
-        <xacro:material_staubli_yellow />
+        <xacro:material_staubli_ral_melon_yellow />
       </visual>
       <collision>
@@ -33,4 +40,11 @@
         </geometry>
       </collision>
+      <inertial>
+          <mass value="45.357763"/>
+          <origin xyz="0.085479 -0.002547 -0.040488" rpy="0.0 0.0 0.0"/>
+          <inertia ixx="0.839141" ixy="0.022637" ixz="0.162457"
+                                  iyy="1.030146" iyz="0.027416"
+                                                 izz="1.064698"/>
+      </inertial>
     </link>
     <link name="${prefix}link_2">
@@ -40,5 +54,5 @@
           <mesh filename="package://staubli_rx160_support/meshes/rx160/visual/link_2.stl"/>
         </geometry>
-        <xacro:material_staubli_yellow />
+        <xacro:material_staubli_ral_melon_yellow />
       </visual>
       <collision>
@@ -48,4 +62,11 @@
         </geometry>
       </collision>
+      <inertial>
+          <mass value="51.266495"/>
+          <origin xyz="-0.000002 0.264164 0.347704" rpy="0.0 0.0 0.0"/>
+          <inertia ixx="5.272800" ixy="0.000010" ixz="0.000017"
+                                  iyy="5.536809" iyz="-0.008261"
+                                                 izz="0.486191"/>
+      </inertial>
     </link>
     <link name="${prefix}link_3">
@@ -55,5 +76,5 @@
           <mesh filename="package://staubli_rx160_support/meshes/rx160/visual/link_3.stl"/>
         </geometry>
-        <xacro:material_staubli_yellow />
+        <xacro:material_staubli_ral_melon_yellow />
       </visual>
       <collision>
@@ -63,4 +84,11 @@
         </geometry>
       </collision>
+      <inertial>
+          <mass value="19.754401"/>
+          <origin xyz="-0.000255 0.016478 -0.003819" rpy="0.0 0.0 0.0"/>
+          <inertia ixx="0.249388" ixy="-0.004901" ixz="0.004825"
+                                  iyy="0.211780"  iyz="0.000574"
+                                                  izz="0.238488"/>
+      </inertial>
     </link>
     <link name="${prefix}link_4">
@@ -70,5 +98,5 @@
           <mesh filename="package://staubli_rx160_support/meshes/rx160/visual/link_4.stl"/>
         </geometry>
-        <xacro:material_staubli_yellow />
+        <xacro:material_staubli_ral_melon_yellow />
       </visual>
       <collision>
@@ -78,4 +106,11 @@
         </geometry>
       </collision>
+      <inertial>
+          <mass value="15.287896"/>
+          <origin xyz="-0.015515 0.000164 0.340348" rpy="0.0 0.0 0.0"/>
+          <inertia ixx="0.331593" ixy="0.000055" ixz="-0.010688"
+                                  iyy="0.320895" iyz="0.000058"
+                                                 izz="0.086557"/>
+      </inertial>
     </link>
     <link name="${prefix}link_5">
@@ -85,5 +120,5 @@
           <mesh filename="package://staubli_rx160_support/meshes/rx160/visual/link_5.stl"/>
         </geometry>
-        <xacro:material_staubli_yellow />
+        <xacro:material_staubli_ral_melon_yellow />
       </visual>
       <collision>
@@ -93,4 +128,11 @@
         </geometry>
       </collision>
+      <inertial>
+          <mass value="0.548088"/>
+          <origin xyz="0.000000 -0.000347 0.023671" rpy="0.0 0.0 0.0"/>
+          <inertia ixx="0.000876" ixy="0.000000" ixz="0.000000"
+                                  iyy="0.000889" iyz="0.000005"
+                                                 izz="0.000412"/>
+      </inertial>
     </link>
     <link name="${prefix}link_6">
@@ -100,5 +142,5 @@
           <mesh filename="package://staubli_rx160_support/meshes/rx160/visual/link_6.stl"/>
         </geometry>
-        <xacro:material_staubli_yellow />
+        <xacro:material_staubli_ral_traffic_grey_b />
       </visual>
       <collision>
@@ -108,4 +150,11 @@
         </geometry>
       </collision>
+      <inertial>
+          <mass value="0.038484"/>
+          <origin xyz="-0.000245 0.000000 -0.007626" rpy="0.0 0.0 0.0"/>
+          <inertia ixx="0.000011" ixy="0.000000" ixz="0.000000"
+                                  iyy="0.000011" iyz="0.000000"
+                                                 izz="0.000021"/>
+      </inertial>
     </link>
     <link name="${prefix}tool0"/>
@@ -116,5 +165,6 @@
       <child link="${prefix}link_1"/>
       <axis xyz="0 0 1"/>
-      <limit lower="-2.967060" upper="2.967060" effort="0" velocity="2.88" />
+      <limit lower="-2.967060" upper="2.967060" effort="692.0" velocity="2.88" />
+      <dynamics damping="0.0" friction="0.0"/>
     </joint>
     <joint name="${prefix}joint_2" type="revolute">
@@ -123,5 +173,6 @@
       <child link="${prefix}link_2"/>
       <axis xyz="0 1 0"/>
-      <limit lower="-2.4" upper="2.4" effort="0" velocity="2.62" />
+      <limit lower="-2.4" upper="2.4" effort="574.0" velocity="2.62" />
+      <dynamics damping="0.0" friction="0.0"/>
     </joint>
     <joint name="${prefix}joint_3" type="revolute">
@@ -130,5 +181,6 @@
       <child link="${prefix}link_3"/>
       <axis xyz="0 1 0"/>
-      <limit lower="-2.62" upper="2.62" effort="0" velocity="3.32" />
+      <limit lower="-2.62" upper="2.62" effort="242.0" velocity="3.32" />
+      <dynamics damping="0.0" friction="0.0"/>
     </joint>
     <joint name="${prefix}joint_4" type="revolute">
@@ -137,5 +189,6 @@
       <child link="${prefix}link_4"/>
       <axis xyz="0 0 1"/>
-      <limit lower="-4.71" upper="4.71" effort="0" velocity="5.15" />
+      <limit lower="-4.71" upper="4.71" effort="58.0" velocity="5.15" />
+      <dynamics damping="0.0" friction="0.0"/>
     </joint>
     <joint name="${prefix}joint_5" type="revolute">
@@ -144,5 +197,9 @@
       <child link="${prefix}link_5"/>
       <axis xyz="0 1 0"/>
-      <limit lower="-1.83" upper="2.09" effort="0" velocity="4.54" />
+      <!-- from Staubli instruction manual:
+      (1) effort limit = 58 Nm if axis 6 torque = 0 Nm
+      (2) effort limit = 29 Nm for maximum torque on axis 6 -->
+      <limit lower="-1.83" upper="2.09" effort="29.0" velocity="4.54" />
+      <dynamics damping="0.0" friction="0.0"/>
     </joint>
     <joint name="${prefix}joint_6" type="revolute">
@@ -151,5 +208,6 @@
       <child link="${prefix}link_6"/>
       <axis xyz="0 0 1"/>
-      <limit lower="-4.71" upper="4.71" effort="0" velocity="7.68" />
+      <limit lower="-4.71" upper="4.71" effort="29.0" velocity="7.68" />
+      <dynamics damping="0.0" friction="0.0"/>
     </joint>
     <joint name="${prefix}joint_6-tool0" type="fixed">

File: staubli_rx160_support/urdf/rx160l.urdf (robot description, URDF)
Before this commit: robot staubli_rx160l, 8 links, 7 joints
Links:
- link base_link: mass None -> 23.085357
- link link_1: mass None -> 45.357763
- link link_2: mass None -> 51.266495
- link link_3: mass None -> 19.754401
- link link_4: mass None -> 27.640019
- link link_5: mass None -> 0.548088
- link link_6: mass None -> 0.038484
Joints:
- joint joint_1: limit lower=-2.967060 upper=2.967060 effort=0 velocity=2.88 -> lower=-2.967060 upper=2.967060 effort=692.0 velocity=2.88
- joint joint_2: limit lower=-2.4 upper=2.4 effort=0 velocity=2.62 -> lower=-2.4 upper=2.4 effort=574.0 velocity=2.62
- joint joint_3: limit lower=-2.62 upper=2.62 effort=0 velocity=3.32 -> lower=-2.62 upper=2.62 effort=242.0 velocity=3.32
- joint joint_4: limit lower=-4.71 upper=4.71 effort=0 velocity=5.15 -> lower=-4.71 upper=4.71 effort=58.0 velocity=5.15
- joint joint_5: limit lower=-1.83 upper=2.09 effort=0 velocity=4.54 -> lower=-1.83 upper=2.09 effort=29.0 velocity=4.54
- joint joint_6: limit lower=-4.71 upper=4.71 effort=0 velocity=7.68 -> lower=-4.71 upper=4.71 effort=29.0 velocity=7.68

File: staubli_rx160_support/urdf/rx160l_macro.xacro (robot description, xacro)
@@ -10,5 +10,5 @@
           <mesh filename="package://staubli_rx160_support/meshes/rx160/visual/base_link.stl"/>
         </geometry>
-        <xacro:material_staubli_yellow />
+        <xacro:material_staubli_ral_melon_yellow />
       </visual>
       <collision>
@@ -18,4 +18,11 @@
         </geometry>
       </collision>
+      <inertial>
+          <mass value="23.085357"/>
+          <origin xyz="0.007579 0.000017 0.180670" rpy="0.0 0.0 0.0"/>
+          <inertia ixx="0.343576" ixy="-0.000062" ixz="-0.002079"
+                                  iyy="0.336217"  iyz="-0.000014"
+                                                  izz="0.334050"/>
+      </inertial>
     </link>
     <link name="${prefix}link_1">
@@ -25,5 +32,5 @@
           <mesh filename="package://staubli_rx160_support/meshes/rx160/visual/link_1.stl"/>
         </geometry>
-        <xacro:material_staubli_yellow />
+        <xacro:material_staubli_ral_melon_yellow />
       </visual>
       <collision>
@@ -33,4 +40,11 @@
         </geometry>
       </collision>
+      <inertial>
+          <mass value="45.357763"/>
+          <origin xyz="0.085479 -0.002547 -0.040488" rpy="0.0 0.0 0.0"/>
+          <inertia ixx="0.839141" ixy="0.022637" ixz="0.162457"
+                                  iyy="1.030146" iyz="0.027416"
+                                                 izz="1.064698"/>
+      </inertial>
     </link>
     <link name="${prefix}link_2">
@@ -40,5 +54,5 @@
           <mesh filename="package://staubli_rx160_support/meshes/rx160/visual/link_2.stl"/>
         </geometry>
-        <xacro:material_staubli_yellow />
+        <xacro:material_staubli_ral_melon_yellow />
       </visual>
       <collision>
@@ -48,4 +62,11 @@
         </geometry>
       </collision>
+      <inertial>
+          <mass value="51.266495"/>
+          <origin xyz="-0.000002 0.264164 0.347704" rpy="0.0 0.0 0.0"/>
+          <inertia ixx="5.272800" ixy="0.000010" ixz="0.000017"
+                                  iyy="5.536809" iyz="-0.008261"
+                                                 izz="0.486191"/>
+      </inertial>
     </link>
     <link name="${prefix}link_3">
@@ -55,5 +76,5 @@
           <mesh filename="package://staubli_rx160_support/meshes/rx160/visual/link_3.stl"/>
         </geometry>
-        <xacro:material_staubli_yellow />
+        <xacro:material_staubli_ral_melon_yellow />
       </visual>
       <collision>
@@ -63,4 +84,11 @@
         </geometry>
       </collision>
+      <inertial>
+          <mass value="19.754401"/>
+          <origin xyz="-0.000255 0.016478 -0.003819" rpy="0.0 0.0 0.0"/>
+          <inertia ixx="0.249388" ixy="-0.004901" ixz="0.004825"
+                                  iyy="0.211780"  iyz="0.000574"
+                                                  izz="0.238488"/>
+      </inertial>
     </link>
     <link name="${prefix}link_4">
@@ -70,5 +98,5 @@
           <mesh filename="package://staubli_rx160_support/meshes/rx160l/visual/link_4.stl"/>
         </geometry>
-        <xacro:material_staubli_yellow />
+        <xacro:material_staubli_ral_melon_yellow />
       </visual>
       <collision>
@@ -78,4 +106,11 @@
         </geometry>
       </collision>
+      <inertial>
+          <mass value="27.640019"/>
+          <origin xyz="-0.009602 0.000028 0.472641" rpy="0.0 0.0 0.0"/>
+          <inertia ixx="1.378080" ixy="0.000062" ixz="-0.042670"
+                                  iyy="1.366754" iyz="0.000069"
+                                                 izz="0.170331"/>
+      </inertial>
     </link>
     <link name="${prefix}link_5">
@@ -85,5 +120,5 @@
           <mesh filename="package://staubli_rx160_support/meshes/rx160/visual/link_5.stl"/>
         </geometry>
-        <xacro:material_staubli_yellow />
+        <xacro:material_staubli_ral_melon_yellow />
       </visual>
       <collision>
@@ -93,4 +128,11 @@
         </geometry>
       </collision>
+      <inertial>
+          <mass value="0.548088"/>
+          <origin xyz="0.000000 -0.000347 0.023671" rpy="0.0 0.0 0.0"/>
+          <inertia ixx="0.000876" ixy="0.000000" ixz="0.000000"
+                                  iyy="0.000889" iyz="0.000005"
+                                                 izz="0.000412"/>
+      </inertial>
     </link>
     <link name="${prefix}link_6">
@@ -100,5 +142,5 @@
           <mesh filename="package://staubli_rx160_support/meshes/rx160/visual/link_6.stl"/>
         </geometry>
-        <xacro:material_staubli_yellow />
+        <xacro:material_staubli_ral_traffic_grey_b />
       </visual>
       <collision>
@@ -108,4 +150,11 @@
         </geometry>
       </collision>
+      <inertial>
+          <mass value="0.038484"/>
+          <origin xyz="-0.000245 0.000000 -0.007626" rpy="0.0 0.0 0.0"/>
+          <inertia ixx="0.000011" ixy="0.000000" ixz="0.000000"
+                                  iyy="0.000011" iyz="0.000000"
+                                                 izz="0.000021"/>
+      </inertial>
     </link>
     <link name="${prefix}tool0"/>
@@ -116,5 +165,6 @@
       <child link="${prefix}link_1"/>
       <axis xyz="0 0 1"/>
-      <limit lower="-2.967060" upper="2.967060" effort="0" velocity="2.88" />
+      <limit lower="-2.967060" upper="2.967060" effort="692.0" velocity="2.88" />
+      <dynamics damping="0.0" friction="0.0"/>
     </joint>
     <joint name="${prefix}joint_2" type="revolute">
@@ -123,5 +173,6 @@
       <child link="${prefix}link_2"/>
       <axis xyz="0 1 0"/>
-      <limit lower="-2.4" upper="2.4" effort="0" velocity="2.62" />
+      <limit lower="-2.4" upper="2.4" effort="574.0" velocity="2.62" />
+      <dynamics damping="0.0" friction="0.0"/>
     </joint>
     <joint name="${prefix}joint_3" type="revolute">
@@ -130,5 +181,6 @@
       <child link="${prefix}link_3"/>
       <axis xyz="0 1 0"/>
-      <limit lower="-2.62" upper="2.62" effort="0" velocity="3.32" />
+      <limit lower="-2.62" upper="2.62" effort="242.0" velocity="3.32" />
+      <dynamics damping="0.0" friction="0.0"/>
     </joint>
     <joint name="${prefix}joint_4" type="revolute">
@@ -137,5 +189,6 @@
       <child link="${prefix}link_4"/>
       <axis xyz="0 0 1"/>
-      <limit lower="-4.71" upper="4.71" effort="0" velocity="5.15" />
+      <limit lower="-4.71" upper="4.71" effort="58.0" velocity="5.15" />
+      <dynamics damping="0.0" friction="0.0"/>
     </joint>
     <joint name="${prefix}joint_5" type="revolute">
@@ -144,5 +197,9 @@
       <child link="${prefix}link_5"/>
       <axis xyz="0 1 0"/>
-      <limit lower="-1.83" upper="2.09" effort="0" velocity="4.54" />
+      <!-- from Staubli instruction manual:
+      (1) effort limit = 58 Nm if axis 6 torque = 0 Nm
+      (2) effort limit = 29 Nm for maximum torque on axis 6 -->
+      <limit lower="-1.83" upper="2.09" effort="29.0" velocity="4.54" />
+      <dynamics damping="0.0" friction="0.0"/>
     </joint>
     <joint name="${prefix}joint_6" type="revolute">
@@ -151,5 +208,6 @@
       <child link="${prefix}link_6"/>
       <axis xyz="0 0 1"/>
-      <limit lower="-4.71" upper="4.71" effort="0" velocity="7.68" />
+      <limit lower="-4.71" upper="4.71" effort="29.0" velocity="7.68" />
+      <dynamics damping="0.0" friction="0.0"/>
     </joint>
     <joint name="${prefix}joint_6-tool0" type="fixed">
